File: KiCad/RippleCharger/WaveformGen.sch (KiCad schematic (older format))
At the start: 50 parts, among them J2 AD9833, Q1 2N3904, U2 LM358, U3 LM358, U4 LM358, U5 LM358, U6 LM358

Commit message: Update PCB layout m include relay footprint, board outlook.Modify Main 0049 code and add CV function
Parts:
- removed Q1: 2N3904, Package_TO_SOT_SMD:SOT-23, symbol Transistor_BJT:2N3904
- removed RY1: RY5W-K, basic:RY5W-K, symbol RippleCharger-rescue:RY5W-K-basic
- added Q1: MMBT3904, Package_TO_SOT_SMD:SOT-23, symbol Transistor_BJT:MMBT3904
- added RY3: RY5W-K, basic:RY5W-K, symbol basic:RY5W-K
- added TP2: base, Connector_PinHeader_2.54mm:PinHeader_1x01_P2.54mm_Vertical, symbol Connector:TestPoint
- D2, D3, D4, D5: footprint Diode_SMD:D_0805_2012Metric_Pad1.15x1.40mm_HandSolder -> Diode_SMD:D_SOD-123
- R23: value 5.6k -> 1k
- TP1: value ac_wave -> Asymm
Connections:
- net +5VD: now also RY3.1
- net GND: now also Q1.2 (E)
- net asymm: now also TP1.1, RY3.8
- net base: now also RV6.1, TP2.1
- net sigRly: now also RY3.4
- net sigout: now also RY3.6
- net at Cs1.1, R2.1, R3.1: no longer TP1.1
- net at R23.2: now also Q1.1 (B)
- net at D5.2 (A): now also Q1.3 (C), RY3.16
- no-connect marks 5 -> 4
Other:
- moved on the sheet: TP1
Changed lines of the file:
@@
 F 0 "D4" H 3250 3683 50  0000 C CNN
 F 1 "1N4148" H 3250 3774 50  0000 C CNN
-F 2 "Diode_SMD:D_0805_2012Metric_Pad1.15x1.40mm_HandSolder" H 3250 3725 50  0001 C CNN
+F 2 "Diode_SMD:D_SOD-123" H 3250 3725 50  0001 C CNN
 F 3 "https://assets.nexperia.com/documents/data-sheet/1N4148_1N4448.pdf" H 3250 3900 50  0001 C CNN
 	1    3250 3900
@@
 F 0 "D2" H 2550 3133 50  0000 C CNN
 F 1 "1N4148" H 2550 3224 50  0000 C CNN
-F 2 "Diode_SMD:D_0805_2012Metric_Pad1.15x1.40mm_HandSolder" H 2550 3175 50  0001 C CNN
+F 2 "Diode_SMD:D_SOD-123" H 2550 3175 50  0001 C CNN
 F 3 "https://assets.nexperia.com/documents/data-sheet/1N4148_1N4448.pdf" H 2550 3350 50  0001 C CNN
 	1    2550 3350
@@
 F 0 "D3" H 3000 4983 50  0000 C CNN
 F 1 "1N4148" H 3000 5074 50  0000 C CNN
-F 2 "Diode_SMD:D_0805_2012Metric_Pad1.15x1.40mm_HandSolder" H 3000 5025 50  0001 C CNN
+F 2 "Diode_SMD:D_SOD-123" H 3000 5025 50  0001 C CNN
 F 3 "https://assets.nexperia.com/documents/data-sheet/1N4148_1N4448.pdf" H 3000 5200 50  0001 C CNN
 	1    3000 5200
@@
 	6500 4950 6550 4950
 Connection ~ 6500 4950
-Wire Wire Line
-	6750 4950 6850 4950
 $Comp
 L Device:R_Small R24
@@
 Wire Wire Line
 	8500 3050 8500 3100
-Wire Wire Line
-	9100 2750 9250 2750
 $Comp
 L power:GND #PWR023
@@
 	-1   0    0    1
 $EndComp
-Text GLabel 6850 4950 2    50   Input ~ 0
+Text GLabel 6950 4950 2    50   Input ~ 0
 asymm
 $Comp
 L Connector:TestPoint TP1
 U 1 1 6168C104
-P 1700 4450
-F 0 "TP1" V 1654 4638 50  0000 L CNN
-F 1 "ac_wave" V 1745 4638 50  0000 L CNN
-F 2 "Connector_PinHeader_2.54mm:PinHeader_1x01_P2.54mm_Vertical" H 1900 4450 50  0001 C CNN
-F 3 "~" H 1900 4450 50  0001 C CNN
-	1    1700 4450
-	0    1    1    0
+P 6850 4950
+F 0 "TP1" V 6804 5138 50  0000 L CNN
+F 1 "Asymm" V 6895 5138 50  0000 L CNN
+F 2 "Connector_PinHeader_2.54mm:PinHeader_1x01_P2.54mm_Vertical" H 7050 4950 50  0001 C CNN
+F 3 "~" H 7050 4950 50  0001 C CNN
+	1    6850 4950
+	1    0    0    -1
 $EndComp
 $Comp
@@
 Text GLabel 9350 5400 2    50   Input ~ 0
 asymm
-Text GLabel 9350 5200 2    50   Input ~ 0
-sigout
 Text GLabel 8300 5300 0    50   Input ~ 0
 sigRly
@@
 AR Path="/6134453E/616E43F3" Ref="R23"  Part="1"
 F 0 "R23" H 8359 4546 50  0000 L CNN
-F 1 "5.6k" H 8359 4455 50  0000 L CNN
+F 1 "1k" H 8359 4455 50  0000 L CNN
 F 2 "Resistor_SMD:R_0805_2012Metric_Pad1.20x1.40mm_HandSolder" H 8300 4500 50  0001 C CNN
 F 3 "~" H 8300 4500 50  0001 C CNN
@@
 	8500 4900 8650 4900
 $Comp
-L Transistor_BJT:2N3904 Q?
-U 1 1 616E4409
-P 8300 4800
-AR Path="/613448A2/616E4409" Ref="Q?"  Part="1"
-AR Path="/6134453E/616E4409" Ref="Q1"  Part="1"
-F 0 "Q1" V 8535 4800 50  0000 C CNN
-F 1 "2N3904" V 8626 4800 50  0000 C CNN
-F 2 "Package_TO_SOT_SMD:SOT-23" H 8500 4725 50  0001 L CIN
-F 3 "https://www.onsemi.com/pub/Collateral/2N3903-D.PDF" H 8300 4800 50  0001 L CNN
-	1    8300 4800
-	0    1    1    0
-$EndComp
-$Comp
 L Diode:1N4148 D?
 U 1 1 616E440F
@@
 F 0 "D5" H 9050 4133 50  0000 C CNN
 F 1 "1N4148" H 9050 4224 50  0000 C CNN
-F 2 "Diode_SMD:D_0805_2012Metric_Pad1.15x1.40mm_HandSolder" H 9050 4175 50  0001 C CNN
+F 2 "Diode_SMD:D_SOD-123" H 9050 4175 50  0001 C CNN
 F 3 "https://assets.nexperia.com/documents/data-sheet/1N4148_1N4448.pdf" H 9050 4350 50  0001 C CNN
 	1    9050 4350
 	-1   0    0    1
-$EndComp
-$Comp
-L RippleCharger-rescue:RY5W-K-basic RY?
-U 1 1 616E4415
-P 9050 5300
-AR Path="/613448A2/616E4415" Ref="RY?"  Part="1"
-AR Path="/6134453E/616E4415" Ref="RY1"  Part="1"
-F 0 "RY1" V 8283 5300 50  0000 C CNN
-F 1 "RY5W-K" V 8374 5300 50  0000 C CNN
-F 2 "basic:RY5W-K" H 9000 5250 50  0001 C CNN
-F 3 "https://www.fcl.fujitsu.com/downloads/MICRO/fcai/relays/ry.pdf" H 9050 5300 50  0001 C CNN
-	1    9050 5300
-	0    1    1    0
 $EndComp
 $Comp
@@
 Text GLabel 9800 4700 1    50   Input ~ 0
 Rly3
-Text GLabel 9250 2750 2    50   Input ~ 0
+Text GLabel 9600 2750 2    50   Input ~ 0
 base
 NoConn ~ 9350 5600
@@
 Wire Wire Line
 	9000 3150 9250 3150
-Wire Wire Line
-	9250 2750 9250 3150
-NoConn ~ 9100 3050
 Wire Wire Line
 	8300 5300 8750 5300
@@
 Wire Wire Line
 	4600 5450 4600 5150
+$Comp
+L Transistor_BJT:MMBT3904 Q1
+U 1 1 61690649
+P 8300 4800
+F 0 "Q1" V 8535 4800 50  0000 C CNN
+F 1 "MMBT3904" V 8626 4800 50  0000 C CNN
+F 2 "Package_TO_SOT_SMD:SOT-23" H 8500 4725 50  0001 L CIN
+F 3 "https://www.onsemi.com/pub/Collateral/2N3903-D.PDF" H 8300 4800 50  0001 L CNN
+	1    8300 4800
+	0    1    1    0
+$EndComp
+$Comp
+L basic:RY5W-K RY3
+U 1 1 616D6B56
+P 9050 5300
+F 0 "RY3" V 8283 5300 50  0000 C CNN
+F 1 "RY5W-K" V 8374 5300 50  0000 C CNN
+F 2 "basic:RY5W-K" H 9000 5250 50  0001 C CNN
+F 3 "https://www.fcl.fujitsu.com/downloads/MICRO/fcai/relays/ry.pdf" H 9050 5300 50  0001 C CNN
+	1    9050 5300
+	0    1    1    0
+$EndComp
+$Comp
+L Connector:TestPoint TP2
+U 1 1 616E9483
+P 9250 2750
+F 0 "TP2" V 9204 2938 50  0000 L CNN
+F 1 "base" V 9295 2938 50  0000 L CNN
+F 2 "Connector_PinHeader_2.54mm:PinHeader_1x01_P2.54mm_Vertical" H 9450 2750 50  0001 C CNN
+F 3 "~" H 9450 2750 50  0001 C CNN
+	1    9250 2750
+	1    0    0    -1
+$EndComp
+Wire Wire Line
+	9100 3050 9250 3050
+Connection ~ 9250 3050
+Wire Wire Line
+	9250 3050 9250 3150
+Wire Wire Line
+	9250 2750 9250 3050
+Wire Wire Line
+	9100 2750 9250 2750
+Connection ~ 9250 2750
+Text GLabel 9350 5200 2    50   Input ~ 0
+sigout
+Wire Wire Line
+	6950 4950 6850 4950
+Wire Wire Line
+	9250 2750 9600 2750
+Wire Wire Line
+	6750 4950 6850 4950
+Connection ~ 6850 4950
 $EndSCHEMATC

Commit message: Fix CV charging route
Parts:
- removed R19, R20: 1k, Resistor_SMD:R_0805_2012Metric_Pad1.20x1.40mm_HandSolder, symbol Device:R_Small
- RV1, RV3: value 20k -> 50k
Connections:
- net 340mV: now also U5.1, U5.2 (-)
Changed lines of the file:
@@
 P 4300 5450
 F 0 "RV1" V 4650 5450 50  0000 C CNN
-F 1 "20k" V 4550 5450 50  0000 C CNN
+F 1 "50k" V 4550 5450 50  0000 C CNN
 F 2 "Potentiometer_THT:Potentiometer_Bourns_3296W_Vertical" H 4300 5450 50  0001 C CNN
 F 3 "~" H 4300 5450 50  0001 C CNN
@@
 	4600 5150 4850 5150
 Connection ~ 4600 5150
-$Comp
-L Amplifier_Operational:LM358 U4
-U 2 1 614F0D30
-P 5800 3750
-F 0 "U4" H 5800 4117 50  0000 C CNN
-F 1 "LM358" H 5800 4026 50  0000 C CNN
-F 2 "Package_SO:SOIC-8_3.9x4.9mm_P1.27mm" H 5800 3750 50  0001 C CNN
-F 3 "http://www.ti.com/lit/ds/symlink/lm2904-n.pdf" H 5800 3750 50  0001 C CNN
-	2    5800 3750
-	1    0    0    -1
-$EndComp
-Text GLabel 5500 3650 0    50   Input ~ 0
-340mV
 $Comp
 L Device:R_Small R11
@@
 	1    0    0    -1
 $EndComp
-Connection ~ 8050 1600
-Wire Wire Line
-	8050 1600 8250 1600
-Wire Wire Line
-	8050 1600 8050 1700
-Wire Wire Line
-	7950 1600 8050 1600
-$Comp
-L power:GND #PWR022
-U 1 1 61529D3B
-P 8050 1900
-F 0 "#PWR022" H 8050 1650 50  0001 C CNN
-F 1 "GND" H 8055 1727 50  0000 C CNN
-F 2 "" H 8050 1900 50  0001 C CNN
-F 3 "" H 8050 1900 50  0001 C CNN
-	1    8050 1900
-	1    0    0    -1
-$EndComp
-$Comp
-L Device:R_Small R20
-U 1 1 61529925
-P 8050 1800
-F 0 "R20" H 7991 1754 50  0000 R CNN
-F 1 "1k" H 7991 1845 50  0000 R CNN
-F 2 "Resistor_SMD:R_0805_2012Metric_Pad1.20x1.40mm_HandSolder" H 8050 1800 50  0001 C CNN
-F 3 "~" H 8050 1800 50  0001 C CNN
-	1    8050 1800
-	-1   0    0    1
-$EndComp
-Connection ~ 7750 1600
-$Comp
-L Device:R_Small R19
-U 1 1 615292B2
-P 7850 1600
-F 0 "R19" V 7654 1600 50  0000 C CNN
-F 1 "1k" V 7745 1600 50  0000 C CNN
-F 2 "Resistor_SMD:R_0805_2012Metric_Pad1.20x1.40mm_HandSolder" H 7850 1600 50  0001 C CNN
-F 3 "~" H 7850 1600 50  0001 C CNN
-	1    7850 1600
-	0    1    1    0
-$EndComp
 Text GLabel 8250 1600 2    50   Input ~ 0
 340mV
@@
 P 6500 1500
 F 0 "RV3" H 6440 1546 50  0000 R CNN
-F 1 "20k" H 6440 1455 50  0000 R CNN
+F 1 "50k" H 6440 1455 50  0000 R CNN
 F 2 "Potentiometer_THT:Potentiometer_Bourns_3296W_Vertical" H 6500 1500 50  0001 C CNN
 F 3 "~" H 6500 1500 50  0001 C CNN
@@
 	6750 4950 6850 4950
 Connection ~ 6850 4950
+Connection ~ 7750 1600
+Wire Wire Line
+	7750 1600 8250 1600
+Text GLabel 5500 3650 0    50   Input ~ 0
+340mV
+$Comp
+L Amplifier_Operational:LM358 U4
+U 2 1 614F0D30
+P 5800 3750
+F 0 "U4" H 5800 4117 50  0000 C CNN
+F 1 "LM358" H 5800 4026 50  0000 C CNN
+F 2 "Package_SO:SOIC-8_3.9x4.9mm_P1.27mm" H 5800 3750 50  0001 C CNN
+F 3 "http://www.ti.com/lit/ds/symlink/lm2904-n.pdf" H 5800 3750 50  0001 C CNN
+	2    5800 3750
+	1    0    0    -1
+$EndComp
 $EndSCHEMATC
